Commit message: 修正urdf限位

File: legged_examples/legged_hunter/legged_hunter_description/urdf/hunter.urdf (robot description, URDF)
Before this commit: robot pai_12dof_v2_0312, 18 links, 17 joints
Joints:
- joint leg_l1_joint: limit lower=-0.5 upper=1.0 effort=21 velocity=21 -> lower=-0.7 upper=0.7 effort=16 velocity=21
- joint leg_l2_joint: limit lower=-0.9 upper=2 effort=21 velocity=21 -> lower=-0.6 upper=0.6 effort=16 velocity=21
- joint leg_l3_joint: limit lower=-0.8 upper=1.8 effort=21 velocity=21 -> lower=-2.0 upper=0.45 effort=16 velocity=21
- joint leg_l4_joint: limit lower=-0.15 upper=2.0 effort=21 velocity=21 -> lower=0 upper=2.0 effort=16 velocity=21
- joint leg_l5_joint: limit lower=-1.57 upper=1.57 effort=21 velocity=21 -> lower=-1.2 upper=0.8 effort=10 velocity=21
- joint leg_r1_joint: limit lower=-1.0 upper=0.5 effort=21 velocity=21 -> lower=-0.7 upper=0.7 effort=16 velocity=21
- joint leg_r2_joint: limit lower=-2 upper=0.9 effort=21 velocity=21 -> lower=-0.6 upper=0.6 effort=16 velocity=21
- joint leg_r3_joint: limit lower=-1.8 upper=0.8 effort=21 velocity=21 -> lower=-2.0 upper=0.45 effort=16 velocity=21
- joint leg_r4_joint: limit lower=-0.15 upper=2.0 effort=21 velocity=21 -> lower=0 upper=2.0 effort=16 velocity=21
- joint leg_r5_joint: limit lower=-1.57 upper=1.57 effort=21 velocity=21 -> lower=-1.2 upper=0.8 effort=10 velocity=21

File: legged_examples/legged_hunter/legged_hunter_description/urdf/hunter_sim.urdf (robot description, URDF)
Before this commit: robot pai_12dof_v2_0312, 18 links, 17 joints
Joints:
- joint leg_l1_joint: limit lower=-0.5 upper=1.0 effort=21 velocity=21 -> lower=-0.7 upper=0.7 effort=16 velocity=21
- joint leg_l2_joint: limit lower=-0.9 upper=2 effort=21 velocity=21 -> lower=-0.6 upper=0.6 effort=16 velocity=21
- joint leg_l3_joint: limit lower=-0.8 upper=1.8 effort=21 velocity=21 -> lower=-2.0 upper=0.45 effort=16 velocity=21
- joint leg_l4_joint: limit lower=-0.15 upper=2.0 effort=21 velocity=21 -> lower=0 upper=2.0 effort=16 velocity=21
- joint leg_l5_joint: limit lower=-0.8 upper=1.2 effort=21 velocity=21 -> lower=-1.2 upper=0.8 effort=10 velocity=21
- joint leg_r1_joint: limit lower=-1.0 upper=0.5 effort=21 velocity=21 -> lower=-0.7 upper=0.7 effort=16 velocity=21
- joint leg_r2_joint: limit lower=-2 upper=0.9 effort=21 velocity=21 -> lower=-0.6 upper=0.6 effort=16 velocity=21
- joint leg_r3_joint: limit lower=-1.8 upper=0.8 effort=21 velocity=21 -> lower=-2.0 upper=0.45 effort=16 velocity=21
- joint leg_r4_joint: limit lower=-0.15 upper=2.0 effort=21 velocity=21 -> lower=0 upper=2.0 effort=16 velocity=21
- joint leg_r5_joint: limit lower=-1.2 upper=0.95 effort=21 velocity=21 -> lower=-1.2 upper=0.8 effort=10 velocity=21

Commit message: 新小Pi仿真能走代码

File: legged_examples/legged_hunter/legged_hunter_description/urdf/hunter.urdf (robot description, URDF)
Before this commit: robot pai_12dof_v2_0312, 18 links, 17 joints
Joints:
- joint leg_l5_fixed_1: origin xyz=0.07 0 -0.010 rpy=0 0 0 -> xyz=0.07 0 -0.01 rpy=0 0 0

File: legged_examples/legged_hunter/legged_hunter_description/urdf/hunter_sim.urdf (robot description, URDF)
Before this commit: robot pai_12dof_v2_0312, 18 links, 17 joints
Joints:
- joint leg_l1_joint: limit lower=-3.14 upper=3.14 effort=21 velocity=21 -> lower=-0.5 upper=1.0 effort=16 velocity=21
- joint leg_l2_joint: limit lower=-3.14 upper=3.14 effort=21 velocity=21 -> lower=-0.9 upper=2 effort=16 velocity=21
- joint leg_l3_joint: limit lower=-3.14 upper=3.14 effort=21 velocity=21 -> lower=-0.8 upper=1.8 effort=16 velocity=21
- joint leg_l4_joint: limit lower=-3.14 upper=3.14 effort=21 velocity=21 -> lower=-0.15 upper=2.0 effort=16 velocity=21
- joint leg_l5_fixed_1: origin xyz=0.07 0 -0.010 rpy=0 0 0 -> xyz=0.07 0 -0.01 rpy=0 0 0
- joint leg_l5_joint: limit lower=-3.14 upper=3.14 effort=21 velocity=21 -> lower=-1.57 upper=1.57 effort=21 velocity=21
- joint leg_r1_joint: limit lower=-3.14 upper=3.14 effort=21 velocity=21 -> lower=-1.0 upper=0.5 effort=16 velocity=21
- joint leg_r2_joint: limit lower=-3.14 upper=3.14 effort=21 velocity=21 -> lower=-2 upper=0.9 effort=16 velocity=21
- joint leg_r3_joint: limit lower=-3.14 upper=3.14 effort=21 velocity=21 -> lower=-1.8 upper=0.8 effort=16 velocity=21
- joint leg_r4_joint: limit lower=-3.14 upper=3.14 effort=21 velocity=21 -> lower=-0.15 upper=2.0 effort=16 velocity=21
- joint leg_r5_joint: limit lower=-3.14 upper=3.14 effort=21 velocity=21 -> lower=-1.57 upper=1.57 effort=21 velocity=21

Commit message: 新小派传统控制5自由度

File: legged_examples/legged_hunter/legged_hunter_description/urdf/hunter.urdf (robot description, URDF)
Before this commit: robot pai_12dof_v2_0312, 18 links, 17 joints
Joints:
- joint leg_l1_joint: limit lower=-3.14 upper=3.14 effort=21 velocity=21 -> lower=-0.6 upper=0.6 effort=16 velocity=21
- joint leg_l2_joint: limit lower=-3.14 upper=3.14 effort=21 velocity=21 -> lower=-0.6 upper=0.6 effort=16 velocity=21
- joint leg_l3_joint: limit lower=-3.14 upper=3.14 effort=21 velocity=21 -> lower=-2.0 upper=0.45 effort=16 velocity=21
- joint leg_l4_joint: limit lower=-3.14 upper=3.14 effort=21 velocity=21 -> lower=0 upper=2.0 effort=16 velocity=21
- joint leg_l5_joint: limit lower=-3.14 upper=3.14 effort=21 velocity=21 -> lower=-1.2 upper=0.8 effort=21 velocity=21
- joint leg_r1_joint: limit lower=-3.14 upper=3.14 effort=21 velocity=21 -> lower=-0.6 upper=0.6 effort=16 velocity=21
- joint leg_r2_joint: limit lower=-3.14 upper=3.14 effort=21 velocity=21 -> lower=-0.6 upper=0.6 effort=16 velocity=21
- joint leg_r3_joint: limit lower=-3.14 upper=3.14 effort=21 velocity=21 -> lower=-2.0 upper=0.45 effort=16 velocity=21
- joint leg_r4_joint: limit lower=-3.14 upper=3.14 effort=21 velocity=21 -> lower=0 upper=2.0 effort=16 velocity=21
- joint leg_r5_joint: limit lower=-3.14 upper=3.14 effort=21 velocity=21 -> lower=-1.2 upper=0.8 effort=21 velocity=21

File: legged_examples/legged_hunter/legged_hunter_description/urdf/hunter_sim.urdf (robot description, URDF)
Before this commit: robot pai_12dof_v2_0312, 18 links, 17 joints
Joints:
- joint leg_l1_joint: limit lower=-0.5 upper=1.0 effort=16 velocity=21 -> lower=-0.6 upper=0.6 effort=16 velocity=21
- joint leg_l2_joint: limit lower=-0.9 upper=2 effort=16 velocity=21 -> lower=-0.6 upper=0.6 effort=16 velocity=21
- joint leg_l3_joint: limit lower=-0.8 upper=1.8 effort=16 velocity=21 -> lower=-2.0 upper=0.45 effort=16 velocity=21
- joint leg_l4_joint: limit lower=-0.15 upper=2.0 effort=16 velocity=21 -> lower=0 upper=2.0 effort=16 velocity=21
- joint leg_l5_joint: limit lower=-1.57 upper=1.57 effort=21 velocity=21 -> lower=-1.2 upper=0.8 effort=21 velocity=21
- joint leg_r1_joint: limit lower=-1.0 upper=0.5 effort=16 velocity=21 -> lower=-0.6 upper=0.6 effort=16 velocity=21
- joint leg_r2_joint: limit lower=-2 upper=0.9 effort=16 velocity=21 -> lower=-0.6 upper=0.6 effort=16 velocity=21
- joint leg_r3_joint: limit lower=-1.8 upper=0.8 effort=16 velocity=21 -> lower=-2.0 upper=0.45 effort=16 velocity=21
- joint leg_r4_joint: limit lower=-0.15 upper=2.0 effort=16 velocity=21 -> lower=0 upper=2.0 effort=16 velocity=21
- joint leg_r5_joint: limit lower=-1.57 upper=1.57 effort=21 velocity=21 -> lower=-1.2 upper=0.8 effort=21 velocity=21
